Commit message: Dev move base (#6)
* added camera urdf and updated rviz config

* Added stereo camera

* simulated realsense d435

* keyboard teleop and documentation

* package.xml dependencies

* modified ekf config and added sensor launch files

* [WIP] Initial creation of the move_base.launch file, which isnt' complete yet

* Added costmap and planner config files, as well as an empty map pair *.yaml/*.pgm

* Replaced some underscores with the correct hyphens in apt install commands package names in root README file

* Changed costmap config to match Husky configs more than the tutorial configs

* Commented AMCL node in the move_base.launch file

* move_base obstacle detection and avoidance

* added clearpath playpen world

* updated rover_gazebo README and rover_nav package.xml

Co-authored-by: philippewarren <philippewarren31@gmail.com>

File: rover_description/urdf/rover.urdf.xacro (robot description, xacro)
@@ -1,5 +1,8 @@
 <?xml version="1.0" ?>
 <robot name="rover" xmlns:xacro="http://ros.org/wiki/xacro">
-   <xacro:arg name="robot_namespace" default="/" />
+  <xacro:include filename="$(find rover_description)/urdf/camera.urdf.xacro"/>
+  <xacro:include filename="$(find rover_description)/urdf/stereo_camera.urdf.xacro"/>
+  <xacro:include filename="$(find rover_description)/urdf/realsense_d435.urdf.xacro" />
+  <xacro:arg name="robot_namespace" default="/" />
   <!-- TODO: adjust geometry-->
   <!-- Base size -->
@@ -61,5 +64,5 @@
   <xacro:macro name="wheel" params="wheel_prefix *joint_pose" >
     <link name="${wheel_prefix}_wheel_link" >
-      <inertial>
+      <inertial>#
         <mass value="2" />
 				<origin xyz="0 0 0" />
@@ -115,4 +118,16 @@
     <origin xyz="${-wheelbase/2} ${-track/2  - wheel_length/2} ${wheel_vertical_offset}" rpy="0 0 0" />
   </xacro:wheel>
+  <!-- Camera -->
+  <xacro:camera_sensor name="camera1" parent="base_link" hfov="1.3962634" image_width="800" image_height="600"  >
+    <origin xyz="0 0 0.5" rpy="0 0 0" />
+  </xacro:camera_sensor>
+  <!-- Stereo camera -->
+  <!--<xacro:stereo_camera_sensor name="stereo_camera" parent="base_link" hfov="1.3962634" image_width="800" image_height="600" camera_distance="0.1" >
+    <origin xyz="${base_x_size/2} 0 0" rpy="0 0 0" />
+  </xacro:stereo_camera_sensor>-->
+  <!-- Intel RealSense d435 -->
+  <xacro:realsense_d435_sensor name="d435" parent="base_link" >
+    <origin xyz="${base_x_size/2} 0 ${base_z_size}" rpy="0 0 0" />
+  </xacro:realsense_d435_sensor>
   <!-- gazebo plugins -->
   <gazebo>
