Commit message: fixed urdf

File: rover_sim/rover_urdf/robot.urdf (robot description, URDF)
Before this commit: robot rover, 7 links, 6 joints
Links:
- link base_urdf: mass 703.12321350783201979 -> 703.12321350783213347; geometry collision mesh filename=package://rover_sim/rover_urdf/base.stl; collision mesh filename=package://rover_sim/rover_urdf/base_urdf.stl
- link j0_urdf: geometry collision mesh filename=package://rover_sim/rover_urdf/j0_urdf.stl; visual mesh filename=package://rover_sim/rover_urdf/j0_urdf.stl
- link j1_urdf: mass 3.5446627968758868121 -> 3.5446627968758885885; geometry collision mesh filename=package://rover_sim/rover_urdf/j1_urdf.stl; visual mesh filename=package://rover_sim/rover_urdf/j1_urdf.stl
- link j2_urdf: mass 1.903643385227656637 -> 1.903643385227656859; geometry collision mesh filename=package://rover_sim/rover_urdf/j2_urdf.stl; visual mesh filename=package://rover_sim/rover_urdf/j2_urdf.stl
- link jlin_urdf: geometry collision mesh filename=package://rover_sim/rover_urdf/jlin_urdf.stl; visual mesh filename=package://rover_sim/rover_urdf/jlin_urdf.stl
- link poignet_rot_urdf: geometry collision mesh filename=package://rover_sim/rover_urdf/poignet_rot_urdf.stl; visual mesh filename=package://rover_sim/rover_urdf/poignet_rot_urdf.stl
- link poignet_ud_urdf: geometry collision mesh filename=package://rover_sim/rover_urdf/poignet_ud_urdf.stl; visual mesh filename=package://rover_sim/rover_urdf/poignet_ud_urdf.stl
Joints:
- joint J0: origin xyz=0 -0.081500000000000016875 -0.055250000000000007438 rpy=-1.570796326794896558 1.4042235959233375642 -6.1196811644548272158e-17 -> xyz=1.3877787807814456755e-16 -0.081500000000000044631 -0.055250000000000076827 rpy=-1.570796326794896558 0.70767284743509584199 -1.667175257035190381e-17
- joint J1: origin xyz=5.5511151231257827021e-17 0.6500000000000000222 -0.077249999999999985345 rpy=3.1415926535897913396 4.5796699765788054391e-15 1.5708019391319063551 -> xyz=5.5511151231257827021e-17 0.65000000000000057732 -0.077250000000000262901 rpy=3.1415926535897926719 -1.1102230246251438447e-16 -1.0209549457332056654
- joint J2: origin xyz=-5.5511151231257827021e-17 0.625 0.043999999999999969691 rpy=9.2703677178582533106e-15 2.9033507699963287332e-16 -2.1679974831754251774 -> xyz=0 0.62500000000000044409 0.043999999999999539479 rpy=7.6620089321465238822e-15 -5.3667135120133940592e-15 -1.7054038722282933715
- joint base_lin: origin xyz=-0.030475478866928244759 0.015999999999999459099 -0.031999999999999889644 rpy=-1.5707963267948972241 -7.4246164771810213122e-16 1.5707963267948958919 -> xyz=0.22341873687837626727 0.0159999999999999587 -0.031999999999999861888 rpy=-1.5707963267948972241 -7.4246164771810203262e-16 1.5707963267948961139
- joint poignet_gd: origin xyz=0.13723394118771259365 -0.066719159564708613308 0.77504773524655989902 rpy=-2.3930394231407654537 -3.8132505453947008231e-16 -1.404223595923336898 -> xyz=0.9461958637762555302 0.35117428972622033445 0.022930263560738683992 rpy=-2.5528968960603362071 -1.883985361725510729e-16 -0.70767284743509584199
- joint poignet_ud: origin xyz=0.021999999999999991784 0 -0.031000000000000138556 rpy=1.5707963267948950037 -1.3457487744925549222 -1.5707963267948812369 -> xyz=0.02199999999999951994 -4.4408920985006261617e-16 -0.030999999999999916511 rpy=-1.570796326794896558 0.17346192190115755638 1.5707963267948901187

Commit message: final forward kin logic

File: rover_sim/rover_urdf/robot.urdf (robot description, URDF)
Before this commit: robot rover, 7 links, 6 joints
Links:
- link base_urdf: mass 703.12321350783213347 -> 703.1232135078319061
- link j1_urdf: mass 3.5446627968758885885 -> 3.5446627968758881444
- link j2_urdf: mass 1.903643385227656859 -> 1.9036433852276570811
- link jlin_urdf: mass 0.57976963990118524084 -> 0.57976963990118512982
Joints:
- joint J0: origin xyz=1.3877787807814456755e-16 -0.081500000000000044631 -0.055250000000000076827 rpy=-1.570796326794896558 0.70767284743509584199 -1.667175257035190381e-17 -> xyz=-1.3877787807814456755e-17 -0.081500000000000044631 -0.055250000000000076827 rpy=-1.570796326794896558 1.5504355345247862186 3.9087839595390209071e-15
- joint J1: origin xyz=5.5511151231257827021e-17 0.65000000000000057732 -0.077250000000000262901 rpy=3.1415926535897926719 -1.1102230246251438447e-16 -1.0209549457332056654 -> xyz=-1.3877787807814456755e-17 0.6500000000000000222 -0.077249999999999985345 rpy=-3.1415926535897908956 -2.6592902268534017048e-15 -0.0013831814381191408301
- joint J2: origin xyz=0 0.62500000000000044409 0.043999999999999539479 rpy=7.6620089321465238822e-15 -5.3667135120133940592e-15 -1.7054038722282933715 -> xyz=3.4694469519536141888e-17 0.62499999999999988898 0.04400000000000003908 rpy=-6.580485871541617736e-15 -1.1990534202759216582e-15 0.044617477012821593618
- joint base_lin: origin xyz=0.22341873687837626727 0.0159999999999999587 -0.031999999999999861888 rpy=-1.5707963267948972241 -7.4246164771810203262e-16 1.5707963267948961139 -> xyz=0.23048828693523157329 0.016000000000000000333 -0.032000000000000000666 rpy=-1.5707963267948970021 2.9143354396410393699e-16 1.5707963267948961139
- joint poignet_gd: limit lower=-3.141592653589793116 upper=3.141592653589793116 effort=1 velocity=20 -> lower=-6.283185307179586232 upper=6.283185307179586232 effort=1 velocity=20; origin xyz=0.9461958637762555302 0.35117428972622033445 0.022930263560738683992 rpy=-2.5528968960603362071 -1.883985361725510729e-16 -0.70767284743509584199 -> xyz=1.5117159709943739365 0.29222822843966539397 -0.035467932922730011081 rpy=1.5707963267948972241 -5.8030238598553389535e-15 1.5707963267948941155
- joint poignet_ud: origin xyz=0.02199999999999951994 -4.4408920985006261617e-16 -0.030999999999999916511 rpy=-1.570796326794896558 0.17346192190115755638 1.5707963267948901187 -> xyz=0.022000000000000075051 0 -0.0310000000000003606 rpy=-1.570796326794896558 -0.0014683454812279856522 1.570796326794891673

Commit message: Final 1

File: rover_sim/rover_urdf/robot.urdf (robot description, URDF)
Before this commit: robot rover, 7 links, 6 joints
Links:
- link j2_urdf: mass 1.9036433852276570811 -> 1.9036433852276564149
- link poignet_rot_urdf: mass 0.48250317769047762484 -> 0.48250317769047756933
Joints:
- joint J0: origin xyz=-1.3877787807814456755e-17 -0.081500000000000044631 -0.055250000000000076827 rpy=-1.570796326794896558 1.5504355345247862186 3.9087839595390209071e-15 -> xyz=0 -0.081500000000000044631 -0.055250000000000021316 rpy=-1.570796326794896558 -1.5707963267701074983 0
- joint J1: origin xyz=-1.3877787807814456755e-17 0.6500000000000000222 -0.077249999999999985345 rpy=-3.1415926535897908956 -2.6592902268534017048e-15 -0.0013831814381191408301 -> xyz=-1.1102230246251565404e-16 0.65000000000000013323 -0.077250000000000040856 rpy=-3.1415926535897926719 4.6444468414471429881e-16 0.67872880729574947001
- joint J2: origin xyz=3.4694469519536141888e-17 0.62499999999999988898 0.04400000000000003908 rpy=-6.580485871541617736e-15 -1.1990534202759216582e-15 0.044617477012821593618 -> xyz=-1.1102230246251565404e-16 0.62500000000000011102 0.043999999999999983569 rpy=-3.9266894517977682624e-15 -8.8941013865064131739e-15 -0.20922196205218601683
- joint base_lin: origin xyz=0.23048828693523157329 0.016000000000000000333 -0.032000000000000000666 rpy=-1.5707963267948970021 2.9143354396410393699e-16 1.5707963267948961139 -> xyz=-0.06385308179254031713 0.016000000000000014211 -0.032000000000000021483 rpy=-1.570796326794896558 2.5673907442389554717e-16 -1.5707963267948958919
- joint poignet_gd: limit lower=-6.283185307179586232 upper=6.283185307179586232 effort=1 velocity=20 -> lower=-3.141592653589793116 upper=3.141592653589793116 effort=1 velocity=20; origin xyz=1.5117159709943739365 0.29222822843966539397 -0.035467932922730011081 rpy=1.5707963267948972241 -5.8030238598553389535e-15 1.5707963267948941155 -> xyz=0.081754356688457471836 1.120967480656651194 -0.16819435518397995999 rpy=-2.6720858083462291077 2.478881469459590623e-11 -1.031381997923065086e-16
- joint poignet_ud: origin xyz=0.022000000000000075051 0 -0.0310000000000003606 rpy=-1.570796326794896558 -0.0014683454812279856522 1.570796326794891673 -> xyz=0.02200000000000001954 2.2204460492503130808e-16 -0.031000000000000249578 rpy=2.0732686826105091365e-17 -1.570796326794891451 0

Commit message: New encoder node + make clean

File: rover_sim/rover_urdf/robot.urdf (robot description, URDF)
Before this commit: robot rover, 7 links, 6 joints
Links:
- link j2_urdf: mass 1.9036433852276564149 -> 1.9036433852276570811
- link poignet_rot_urdf: mass 0.48250317769047756933 -> 0.48250317769047762484
Joints:
- joint J0: origin xyz=0 -0.081500000000000044631 -0.055250000000000021316 rpy=-1.570796326794896558 -1.5707963267701074983 0 -> xyz=-1.3877787807814456755e-17 -0.081500000000000044631 -0.055250000000000076827 rpy=-1.570796326794896558 1.5504355345247862186 3.9087839595390209071e-15
- joint J1: origin xyz=-1.1102230246251565404e-16 0.65000000000000013323 -0.077250000000000040856 rpy=-3.1415926535897926719 4.6444468414471429881e-16 0.67872880729574947001 -> xyz=-1.3877787807814456755e-17 0.6500000000000000222 -0.077249999999999985345 rpy=-3.1415926535897908956 -2.6592902268534017048e-15 -0.0013831814381191408301
- joint J2: origin xyz=-1.1102230246251565404e-16 0.62500000000000011102 0.043999999999999983569 rpy=-3.9266894517977682624e-15 -8.8941013865064131739e-15 -0.20922196205218601683 -> xyz=3.4694469519536141888e-17 0.62499999999999988898 0.04400000000000003908 rpy=-6.580485871541617736e-15 -1.1990534202759216582e-15 0.044617477012821593618
- joint base_lin: origin xyz=-0.06385308179254031713 0.016000000000000014211 -0.032000000000000021483 rpy=-1.570796326794896558 2.5673907442389554717e-16 -1.5707963267948958919 -> xyz=0.23048828693523157329 0.016000000000000000333 -0.032000000000000000666 rpy=-1.5707963267948970021 2.9143354396410393699e-16 1.5707963267948961139
- joint poignet_gd: limit lower=-3.141592653589793116 upper=3.141592653589793116 effort=1 velocity=20 -> lower=-6.283185307179586232 upper=6.283185307179586232 effort=1 velocity=20; origin xyz=0.081754356688457471836 1.120967480656651194 -0.16819435518397995999 rpy=-2.6720858083462291077 2.478881469459590623e-11 -1.031381997923065086e-16 -> xyz=1.5117159709943739365 0.29222822843966539397 -0.035467932922730011081 rpy=1.5707963267948972241 -5.8030238598553389535e-15 1.5707963267948941155
- joint poignet_ud: origin xyz=0.02200000000000001954 2.2204460492503130808e-16 -0.031000000000000249578 rpy=2.0732686826105091365e-17 -1.570796326794891451 0 -> xyz=0.022000000000000075051 0 -0.0310000000000003606 rpy=-1.570796326794896558 -0.0014683454812279856522 1.570796326794891673
