Commit message: Rover fully spawned in rvis

File: rover_sim/model/rover.urdf (robot description, URDF)
Before this commit: robot rover, 7 links, 6 joints
Links:
- added link ARM_BASE, mass 0.512622788118868; collision mesh filename=package://rover_sim/meshes/ARM_BASE.STL; visual mesh filename=package://rover_sim/meshes/ARM_BASE.STL
- added link J0, mass 0.14826651920567; collision mesh filename=package://rover_sim/meshes/J0.STL; visual mesh filename=package://rover_sim/meshes/J0.STL
- added link J1, mass 0.874667906519395; collision mesh filename=package://rover_sim/meshes/J1.STL; visual mesh filename=package://rover_sim/meshes/J1.STL
- added link J2, mass 1.96312360277631; collision mesh filename=package://rover_sim/meshes/J2.STL; visual mesh filename=package://rover_sim/meshes/J2.STL
- added link J3, mass 1.8167140049107; collision mesh filename=package://rover_sim/meshes/J3.STL; visual mesh filename=package://rover_sim/meshes/J3.STL
- added link J4, mass 0.132606093266041; collision mesh filename=package://rover_sim/meshes/J4.STL; visual mesh filename=package://rover_sim/meshes/J4.STL
- added link J5, mass 0.458653210732393; collision mesh filename=package://rover_sim/meshes/J5.STL; visual mesh filename=package://rover_sim/meshes/J5.STL
- link ROCKER_L: geometry collision mesh filename=package://rover_sim/meshes/ROCKER_L.STL; visual mesh filename=package://rover_sim/meshes/ROCKER_L.STL
- link ROCKER_R: geometry collision mesh filename=package://rover_sim/meshes/ROCKER_R.STL; visual mesh filename=package://rover_sim/meshes/ROCKER_R.STL
- link WHEEL_FL: geometry collision mesh filename=package://rover_sim/meshes/WHEEL_FL.STL; visual mesh filename=package://rover_sim/meshes/WHEEL_FL.STL
- link WHEEL_FR: geometry collision mesh filename=package://rover_sim/meshes/WHEEL_FR.STL; visual mesh filename=package://rover_sim/meshes/WHEEL_FR.STL
- link WHEEL_RL: geometry collision mesh filename=package://rover_sim/meshes/WHEEL_RL.STL; visual mesh filename=package://rover_sim/meshes/WHEEL_RL.STL
- link WHEEL_RR: geometry collision mesh filename=package://rover_sim/meshes/WHEEL_RR.STL; visual mesh filename=package://rover_sim/meshes/WHEEL_RR.STL
- link base_link: geometry collision mesh filename=package://rover_sim/meshes/base_link.STL; visual mesh filename=package://rover_sim/meshes/base_link.STL
Joints:
- added joint ARM_BASE_JOINT: type fixed, parent base_link, child ARM_BASE, origin xyz=0.11285 -0.53465 0.32484 rpy=1.5708 0 0, axis 0 0 0
- added joint J0_JOINT: type prismatic, parent ARM_BASE, child J0, origin xyz=-0.28085 0 0 rpy=0 0 0, axis 1 0 0, limit lower=-3.14 upper=3.14 effort=300 velocity=3
- added joint J1_JOINT: type revolute, parent J0, child J1, origin xyz=0 0 0 rpy=3.1416 0 3.1416, axis 0 1 0, limit lower=-3.14 upper=3.14 effort=300 velocity=3
- added joint J2_JOINT: type revolute, parent J1, child J2, origin xyz=0 0.06065 0 rpy=0 0 0, axis 1 0 0, limit lower=-3.14 upper=3.14 effort=300 velocity=3
- added joint J3_JOINT: type revolute, parent J2, child J3, origin xyz=0 0.65 0 rpy=0 0 0, axis 1 0 0, limit lower=-3.14 upper=3.14 effort=300 velocity=3
- added joint J4_JOINT: type revolute, parent J3, child J4, origin xyz=0 0.625 0 rpy=3.1416 0 3.1416, axis 1 0 0, limit lower=-3.14 upper=3.14 effort=300 velocity=3
- added joint J5_JOINT: type revolute, parent J4, child J5, origin xyz=0 0.0455 0 rpy=0 0 0, axis 0 1 0, limit lower=-3.14 upper=3.14 effort=300 velocity=3

Commit message: rover spawn in gz and rviz

File: rover_sim/model/rover.urdf (robot description, URDF)
Before this commit: robot rover, 14 links, 13 joints
Links:
- link ARM_BASE: geometry collision mesh filename=model://rover_sim/meshes/ARM_BASE.STL; visual mesh filename=model://rover_sim/meshes/ARM_BASE.STL
- link J0: geometry collision mesh filename=model://rover_sim/meshes/J0.STL; visual mesh filename=model://rover_sim/meshes/J0.STL
- link J1: geometry collision mesh filename=model://rover_sim/meshes/J1.STL; visual mesh filename=model://rover_sim/meshes/J1.STL
- link J2: geometry collision mesh filename=model://rover_sim/meshes/J2.STL; visual mesh filename=model://rover_sim/meshes/J2.STL
- link J3: geometry collision mesh filename=model://rover_sim/meshes/J3.STL; visual mesh filename=model://rover_sim/meshes/J3.STL
- link J4: geometry collision mesh filename=model://rover_sim/meshes/J4.STL; visual mesh filename=model://rover_sim/meshes/J4.STL
- link J5: geometry collision mesh filename=model://rover_sim/meshes/J5.STL; visual mesh filename=model://rover_sim/meshes/J5.STL
- link ROCKER_L: geometry collision mesh filename=model://rover_sim/meshes/ROCKER_L.STL; visual mesh filename=model://rover_sim/meshes/ROCKER_L.STL
- link ROCKER_R: geometry collision mesh filename=model://rover_sim/meshes/ROCKER_R.STL; visual mesh filename=model://rover_sim/meshes/ROCKER_R.STL
- link WHEEL_FL: geometry collision mesh filename=model://rover_sim/meshes/WHEEL_FL.STL; visual mesh filename=model://rover_sim/meshes/WHEEL_FL.STL
- link WHEEL_FR: geometry collision mesh filename=model://rover_sim/meshes/WHEEL_FR.STL; visual mesh filename=model://rover_sim/meshes/WHEEL_FR.STL
- link WHEEL_RL: geometry collision mesh filename=model://rover_sim/meshes/WHEEL_RL.STL; visual mesh filename=model://rover_sim/meshes/WHEEL_RL.STL
- link WHEEL_RR: geometry collision mesh filename=model://rover_sim/meshes/WHEEL_RR.STL; visual mesh filename=model://rover_sim/meshes/WHEEL_RR.STL
- link base_link: geometry collision mesh filename=model://rover_sim/meshes/base_link.STL; visual mesh filename=model://rover_sim/meshes/base_link.STL
