Commit message: Moving in gz w/ ccmd_vel topic

File: rover_sim/description/rover_core.xacro (robot description, xacro)
@@ -1,4 +1,13 @@
 <?xml version="1.0"?>
-<robot name="rover">
+<robot xmlns:xacro="http://www.ros.org/wiki/xacro">
+    <material name="forest_green">
+        <color rgba="0.13 0.55 0.13 1"/>
+    </material>
+    <material name="grey">
+        <color rgba="0.5 0.5 0.5 1"/>
+    </material>
+    <material name="black">
+        <color rgba="0 0 0 1"/>
+    </material>
     <link name="base_link">
         <inertial>
@@ -23,4 +32,7 @@
         </collision>
     </link>
+    <gazebo reference="base_link">
+        <material>Gazebo/forest_green</material>
+    </gazebo>
     <link name="ROCKER_L">
         <inertial>
@@ -45,4 +57,7 @@
         </collision>
     </link>
+    <gazebo reference="ROCKER_L">
+        <material>Gazebo/grey</material>
+    </gazebo>
     <link name="ROCKER_R">
         <inertial>
@@ -67,4 +82,7 @@
         </collision>
     </link>
+    <gazebo reference="ROCKER_R">
+        <material>Gazebo/grey</material>
+    </gazebo>
     <link name="WHEEL_FL">
         <inertial>
@@ -89,4 +107,7 @@
         </collision>
     </link>
+    <gazebo reference="WHEEL_FL">
+        <material>Gazebo/black</material>
+    </gazebo>
     <link name="WHEEL_RL">
         <inertial>
@@ -111,4 +132,7 @@
         </collision>
     </link>
+    <gazebo reference="WHEEL_RL">
+        <material>Gazebo/black</material>
+    </gazebo>
     <link name="WHEEL_FR">
         <inertial>
@@ -132,5 +156,8 @@
             </geometry>
         </collision>
-    </link>
+    </link>]
+    <gazebo reference="WHEEL_FR">
+        <material>Gazebo/black</material>
+    </gazebo>
     <link name="WHEEL_RR">
         <inertial>
@@ -155,4 +182,7 @@
         </collision>
     </link>
+    <gazebo reference="WHEEL_RR">
+        <material>Gazebo/black</material>
+    </gazebo>
     <joint name="ROCKER_L_JOINT" type="revolute">
         <origin xyz="0.3766 -0.20681 0.078821" rpy="1.5708 0 1.5708" />
@@ -197,24 +227,3 @@
         <limit lower="100" upper="100" effort="0" velocity="20" />
     </joint>
-    <gazebo>
-        <plugin filename="libignition-gazebo-diff-drive-system.so" name="ignition::gazebo::systems::DiffDrive">
-            <left_joint>WHEEL_FL_JOINT</left_joint>
-            <!-- <left_joint>WHEEL_RL_JOINT</left_joint> -->
-            <right_joint>WHEEL_FR_JOINT</right_joint>
-            <!-- <right_joint>WHEEL_RR_JOINT</right_joint> -->
-            <wheel_separation>0.65290</wheel_separation>
-            <wheel_radius>0.27200</wheel_radius>
-            <!-- Limits -->
-            <!-- <max_wheel_torque>200</max_wheel_torque> -->
-            <max_linear_acceleration>0.33</max_linear_acceleration>
-            <!-- Input -->
-            <topic>cmd_vel</topic>
-            <!-- Output -->
-            <frame_id>odom</frame_id>
-            <child_frame_id>base_link</child_frame_id>
-            <odom_topic>odom</odom_topic>
-            <odom_publisher_frequency>30</odom_publisher_frequency>
-            <tf_topic>/tf</tf_topic>
-        </plugin>
-    </gazebo>
 </robot>
